Commit message: update urdf

File: src/manipulator_6dof_description/urdf/manipulator.urdf (robot description, URDF)
Before this commit: robot manipulator, 8 links, 7 joints
Links:
- removed link link_1
- removed link link_2
- removed link link_3
- removed link link_4
- removed link link_5
- removed link link_6
- added link link_1_1, mass 1.044429977886197; collision mesh filename=package://manipulator_6dof_description/meshes/link_1_1.stl scale=0.001 0.001 0.001; visual mesh filename=package://manipulator_6dof_description/meshes/link_1_1.stl scale=0.001 0.001 0.001
- added link link_2_1, mass 1.0723019224070052; collision mesh filename=package://manipulator_6dof_description/meshes/link_2_1.stl scale=0.001 0.001 0.001; visual mesh filename=package://manipulator_6dof_description/meshes/link_2_1.stl scale=0.001 0.001 0.001
- added link link_3_1, mass 0.8938660668299434; collision mesh filename=package://manipulator_6dof_description/meshes/link_3_1.stl scale=0.001 0.001 0.001; visual mesh filename=package://manipulator_6dof_description/meshes/link_3_1.stl scale=0.001 0.001 0.001
- added link link_4_1, mass 0.8311251067189291; collision mesh filename=package://manipulator_6dof_description/meshes/link_4_1.stl scale=0.001 0.001 0.001; visual mesh filename=package://manipulator_6dof_description/meshes/link_4_1.stl scale=0.001 0.001 0.001
- added link link_5_1, mass 0.8431959857300293; collision mesh filename=package://manipulator_6dof_description/meshes/link_5_1.stl scale=0.001 0.001 0.001; visual mesh filename=package://manipulator_6dof_description/meshes/link_5_1.stl scale=0.001 0.001 0.001
- added link link_6_1, mass 0.08319729963947381; collision mesh filename=package://manipulator_6dof_description/meshes/link_6_1.stl scale=0.001 0.001 0.001; visual mesh filename=package://manipulator_6dof_description/meshes/link_6_1.stl scale=0.001 0.001 0.001
- link base_link: mass 3.082687791334984 -> 2.1649980446638213
Joints:
- joint revolute1: child link_1 -> link_1_1; origin xyz=0.0 0.0 0.05 rpy=0 0 0 -> xyz=0.0 0.0 0.062 rpy=0 0 0
- joint revolute2: child link_2 -> link_2_1; origin xyz=-0.03 0.0 0.1 rpy=0 0 0 -> xyz=-0.025 0.0002 0.054 rpy=0 0 0; parent link_1 -> link_1_1
- joint revolute3: axis 1.0 0.0 0.0 -> 1.0 -0.0 0.0; child link_3 -> link_3_1; origin xyz=0.0 0.2 0.0 rpy=0 0 0 -> xyz=0.0 0.0002 0.105 rpy=0 0 0; parent link_2 -> link_2_1
- joint revolute4: axis 0.0 1.0 0.0 -> -0.0 0.0 1.0; child link_4 -> link_4_1; origin xyz=0.03 0.1 0.0 rpy=0 0 0 -> xyz=0.025 0.0 0.08 rpy=0 0 0; parent link_3 -> link_3_1
- joint revolute5: child link_5 -> link_5_1; origin xyz=0.025 0.05 0.0 rpy=0 0 0 -> xyz=0.025 0.0 0.053 rpy=0 0 0; parent link_4 -> link_4_1
- joint revolute6: axis 0.0 1.0 0.0 -> -0.0 -0.0 1.0; child link_6 -> link_6_1; origin xyz=-0.03 0.05 0.0 rpy=0 0 0 -> xyz=-0.025 0.0002 0.093 rpy=0 0 0; parent link_5 -> link_5_1
